File: PCB/fumebuddy.kicad_pcb (KiCad board)
At the start: 2 copper layers, 26.2 x 67.2 mm, 24 parts, among them J1 USB_B_Micro, J2 STATION, J3 FTDI, SW1 SW_SPDT, SW2 SW_SPDT, SW4 SW_OPT, U1 AP7361C-33E, U2 CPC1017N (NO), U4 ESP32-WROOM-32D, U5 CPC1117N (NC)

Commit message: v5
Parts:
- removed R9: 100k, Resistor_SMD:R_1206_3216Metric
- added R6: 100k, Resistor_SMD:R_1206_3216Metric, F.Cu at (138.5, 100.4)
- J3: value FTDI -> esp32buddy; footprint !Custom:FTDI-3Pin -> !Greg:esp32buddy-2.54mm
- R1, R2, R4: value 4.7k -> 4k7
- SW3: renamed from FLASH; footprint Button_Switch_SMD:SW_SPST_PTS810 -> Connector_PinHeader_2.54mm:PinHeader_1x02_P2.54mm_Vertical
- moved REF** 19.9 mm to (127.5, 91.5)
- moved J3 17.5 mm to (133.5, 102.0), turned to 180 degrees
Connections:
- J1 pad 2: Net-(J1-Pad2) -> (no net)
- J1 pad 3: Net-(J1-Pad3) -> (no net)
- J1 pad 4: Net-(J1-Pad4) -> (no net)
- J2 pad S: Net-(J2-PadS) -> (no net)
- J3 pad 1: /RXD -> GND
- J3 pad 2: GND -> /TXD
- J3 pad 3: /TXD -> /RXD
- SW1 pad 3: Net-(SW1-Pad3) -> (no net)
- SW2 pad 3: Net-(SW2-Pad3) -> (no net)
- SW3 pad 1: Net-(R9-Pad1) -> /GPIO0
- U4 pad 12: Net-(U4-Pad12) -> (no net)
- U4 pad 13: /RELAY_AUX -> (no net)
- U4 pad 16: Net-(U4-Pad16) -> (no net)
- U4 pad 17: Net-(U4-Pad17) -> (no net)
- U4 pad 18: Net-(U4-Pad18) -> (no net)
- U4 pad 19: Net-(U4-Pad19) -> (no net)
- U4 pad 20: Net-(U4-Pad20) -> (no net)
- U4 pad 21: Net-(U4-Pad21) -> (no net)
- U4 pad 22: Net-(U4-Pad22) -> (no net)
- U4 pad 23: Net-(U4-Pad23) -> (no net)
- U4 pad 24: Net-(U4-Pad24) -> /SENSOR
- U4 pad 25: Net-(R9-Pad1) -> /GPIO0
- U4 pad 26: Net-(U4-Pad26) -> (no net)
- U4 pad 27: Net-(U4-Pad27) -> (no net)
- U4 pad 28: /SENSOR -> (no net)
- U4 pad 3: +3V3 -> /EN
- U4 pad 30: Net-(U4-Pad30) -> (no net)
- U4 pad 31: Net-(U4-Pad31) -> (no net)
- U4 pad 32: Net-(U4-Pad32) -> (no net)
- U4 pad 33: Net-(U4-Pad33) -> (no net)
- U4 pad 36: Net-(U4-Pad36) -> (no net)
- U4 pad 37: Net-(U4-Pad37) -> (no net)
- U4 pad 39: (no net) -> GND
- U4 pad 4: Net-(U4-Pad4) -> (no net)
- U4 pad 5: Net-(U4-Pad5) -> (no net)
- U4 pad 6: Net-(U4-Pad6) -> (no net)
- U4 pad 7: Net-(U4-Pad7) -> (no net)
- U4 pad 8: Net-(U4-Pad8) -> (no net)
- U4 pad 9: Net-(U4-Pad9) -> (no net)
Routing:
- net Net-(R9-Pad1): track 51.8 -> 0.00 mm, vias 2 -> 0
- net /GPIO0: track 0.00 -> 44.4 mm, vias 0 -> 2
- net Net-(SW1-Pad1): track 34.8 -> 0.35 mm, vias 3 -> 0
- net /EN: track 0.00 -> 30.8 mm, vias 0 -> 4
- net Net-(J2-PadT): track 46.0 -> 26.9 mm, vias 5 -> 4
- net /RXD: track 9.99 -> 0.00 mm, vias 1 -> 0
- net /SENSOR: track 4.05 -> 0.00 mm
- net /TXD: track 13.8 -> 11.3 mm
- net Net-(R1-Pad2): track 66.2 -> 68.2 mm
- net Net-(R4-Pad2): track 60.4 -> 62.1 mm
- net +3V3: track 57.6 -> 58.9 mm, vias 2 -> 3
- net GND: track 25.6 -> 26.2 mm
Other:
- board text added: "fumebuddy v5"
- board text removed: "fumebuddy v4"

Commit message: v5 final sent to fab
Parts:
- removed SW4: SW_OPT, Connector_PinHeader_2.54mm:PinHeader_1x02_P2.54mm_Vertical
- added J4: TOUCH, Connector_PinHeader_2.54mm:PinHeader_1x01_P2.54mm_Vertical, B.Cu at (129.8, 109.5)
- moved J3 1.25 mm to (134.8, 102.0)
- moved SW3 1.04 mm to (131.0, 134.0)
Connections:
- J3 pad 4: (no net) -> +3V3
- U4 pad 10: Net-(SW4-Pad1) -> (no net)
- U4 pad 24: /SENSOR -> /TOUCH
- U4 pad 30: (no net) -> /SENSOR
Routing:
- net Net-(SW4-Pad1): track 66.9 -> 0.00 mm, vias 2 -> 0
- net Net-(J2-PadT): track 26.9 -> 53.8 mm, vias 4 -> 6
- net /RXD: track 0.00 -> 22.7 mm, vias 0 -> 1
- net Net-(SW1-Pad1): track 0.35 -> 21.6 mm
- net /EN: track 30.8 -> 45.5 mm, vias 4 -> 5
- net /TXD: track 11.3 -> 20.9 mm
- net /TOUCH: track 0.00 -> 8.77 mm
- net /GPIO0: track 44.4 -> 51.3 mm
- net +3V3: track 58.9 -> 62.7 mm, vias 3 -> 4
- net /SENSOR: track 0.00 -> 3.37 mm
- net VBUS: track 50.5 -> 49.7 mm
- net GND: vias 15 -> 13
Other:
- outline, holes or cut-outs redrawn
- board text added: "HIDE ME"
